Commit message: this is for the gazebo

File: robot_parts/description/robot_core.xacro (robot description, xacro)
@@ -41,4 +41,7 @@
         </xacro:inertial_box>
     </link>
+    <gazebo reference="chassis">
+        <material>Gazebo/White</material>
+    </gazebo>
     <joint name="left_wheel_joint" type="continuous">
         <parent link="base_link"/>
@@ -65,4 +68,7 @@
         </xacro:inertial_cylinder>
         </link>
+    <gazebo reference="left_wheel">
+        <material>Gazebo/Blue</material>
+    </gazebo>
         <joint name="right_wheel_joint" type="continuous">
         <parent link="base_link"/>
@@ -89,4 +95,7 @@
         </xacro:inertial_cylinder>
         </link>
+    <gazebo reference="right_wheel">
+        <material>Gazebo/Blue</material>
+    </gazebo>
         <!-- caster wheel link-->
         <joint name="caster_wheel_joint" type="fixed">
@@ -111,3 +120,8 @@
             </xacro:inertial_sphere>
         </link>
+    <gazebo reference="caster_wheel">
+        <material>Gazebo/Black</material>
+        <mu1 value="0.001"/>
+        <mu2 value="0.001"/>
+    </gazebo>
 </robot>

File: robot_parts/description/two_wheeled_robot.xacro (robot description, xacro)
@@ -2,3 +2,4 @@
 <robot name="two_wheeled_robot" xmlns:xacro="http://www.ros.org/wiki/xacro">
     <xacro:include filename="robot_core.xacro"/>
+    <xacro:include filename="gazebo_control.xacro"/>
 </robot>

Commit message: added yaml and ros2 control xacro files

File: robot_parts/description/robot_core.xacro (robot description, xacro)
@@ -11,6 +11,9 @@
         <color rgba="0.2 0.2 1 1"/>
     </material>
-        <material name="black">
+    <material name="black">
         <color rgba="0 0 0 1"/>
+    </material>
+    <material name="Red">
+        <color rgba="1 0 0 1"/>
     </material>
     <!--Base link-->
